File: USB HUB.kicad_sch (KiCad schematic)
At the start: 0 parts

Commit message: First Major Update of 2023
Major updates to schematics and first revisions of PCB layout
Parts:
- added C? (x8): 100n, Capacitor_SMD:C_0603_1608Metric, symbol Device:C
- added C? (x3): 1u, Capacitor_SMD:C_0603_1608Metric, symbol Device:C
- added C?: 10u, Capacitor_SMD:C_0603_1608Metric, symbol Device:C
- added F? (x3): 500mA, josh-passives-smt:Fuse_0805_2012Metric, symbol Device:Polyfuse
- added FB? (x4): 600R, josh-passives-smt:Ferrite_Bead_0603, symbol josh-passive:Ferrite_Bead_PWR
- added J? (x3): USB_C_Receptacle_USB2.0, Connector_USB:USB_C_Receptacle_HRO_TYPE-C-31-M-12, symbol Connector:USB_C_Receptacle_USB2.0
- added J? (x2): SM04B-SRSS-TB(LF)(SN), random-keyboard-parts:JST-SR-4, symbol Connector_Generic:Conn_01x04
- added U? (x3): USBLC6-2SC6, Package_TO_SOT_SMD:SOT-23-6, symbol josh-ic:USBLC6-2SC6
Connections:
- new net: C?.1, F?.1, J?.A4 (VBUS), J?.A9 (VBUS), J?.B4 (VBUS), J?.B9 (VBUS), U?.5 (VBUS) (x3)
- new net: F?.2, FB?.1 (x3)
- new net: J?.A6 (D+), J?.B6 (D+), U?.3 (IO2) (x3)
- new net: J?.A7 (D-), J?.B7 (D-), U?.1 (IO1) (x3)
- new net +3.3VA: C?.1, C?.1, C?.1, C?.1, C?.1, C?.1, FB?.1
- new net +3V3: C?.1, C?.1, C?.1, FB?.2
- new net +5V: FB?.2, FB?.2, FB?.2
- new net D1_D+: U?.4 (IO2)
- new net D1_D-: U?.6 (IO1)
- new net D2_D+: U?.4 (IO2)
- new net D2_D-: U?.6 (IO1)
- new net D3_D+: U?.4 (IO2)
- new net D3_D-: U?.6 (IO1)
- new net DN: J?.2 (Pin_2), J?.2 (Pin_2)
- new net DP: J?.3 (Pin_3), J?.3 (Pin_3)
- new net GND: C?.2, C?.2, C?.2, C?.2, C?.2, C?.2, C?.2, C?.2, C?.2, C?.2, C?.2, C?.2, J?.4 (Pin_4), J?.4 (Pin_4), J?.A1 (GND), J?.A1 (GND), J?.A1 (GND), J?.A12 (GND), J?.A12 (GND), J?.A12 (GND), J?.B1 (GND), J?.B1 (GND), J?.B1 (GND), J?.B12 (GND), J?.B12 (GND), J?.B12 (GND), J?.S1 (SHIELD), J?.S1 (SHIELD), J?.S1 (SHIELD), U?.2 (GND), U?.2 (GND), U?.2 (GND)
- new net VCC: J?.1 (Pin_1), J?.1 (Pin_1)
- no-connect marks 0 -> 12
Other:
- note added: "D2"
- note added: "D3"
- note added: "Downstream Ports - D1"
- note added: "USB Hub Power"
