File: unified port.kicad_sch (KiCad schematic)
At the start: 23 parts

Commit message: First Major Update of 2023
Major updates to schematics and first revisions of PCB layout
Parts:
- removed D? (x2): PMEG2010AEB, Bonsai_C4:D_SOD-523, symbol Bonsai_C4:PMEG2010AEB
- removed D?: SMF5.0A, Bonsai_C4:D_SOD-123FL, symbol Bonsai_C4:SMF5.0A
- removed F?: SMD-PPTC-500MA_0805_, Bonsai_C4:F0805, symbol Bonsai_C4:SMD-PPTC-500MA_0805_
- removed FB?: fb_0402_26ohm, Bonsai_C4:R_0402_1005Metric, symbol Bonsai_C4:fb_0402_26ohm
- removed J?: MC-311D, Bonsai_C4:MC-311D, symbol Bonsai_C4:MC-311D
- removed R? (x2): r_5.1k_0402_1p, Bonsai_C4:R_0402_1005Metric, symbol Bonsai_C4:r_5.1k_0402_1p
- removed U?: TPD4E05U06DQAR, acheron_Components:USON-10_2.5x1.0mm_P0.5mm, symbol Unified-Daughterboard-rescue:TPD4E05U06DQAR-acheronSymbols
- removed U?: SRV05-4, Bonsai_C4:SOT-23-6, symbol Bonsai_C4:SRV05-4
- added U8: USBLC6-2SC6, Package_TO_SOT_SMD:SOT-23-6, symbol josh-ic:USBLC6-2SC6
- gave numbers to parts that had none: 13
Connections:
- net D+: now also J6.A6 (D+), J6.B6 (D+), U8.3 (IO2)
- net D-: now also J6.A7 (D-), J6.B7 (D-), U8.1 (IO1)
- net GNDPWR: now also U8.2 (GND)
- net VBUS: now also U8.5 (VBUS)
- removed net DA+: J6.A6 (D+), J6.B6 (D+), J7.3 (Pin_3)
- removed net DA-: J6.A7 (D-), J6.B7 (D-), J7.2 (Pin_2)
- new net DN: J7.2 (Pin_2), U8.6 (IO1)
- new net DP: J7.3 (Pin_3), U8.4 (IO2)
- no-connect marks 4 -> 5
Other:
- note removed: "To LDO"
- moved on the sheet: J6, L1, MH1, MH2, MH3, MH4, R10, R11
