File: The-GarlicBoard-2.kicad_pcb (KiCad board)
At the start: 2 copper layers, 365.9 x 80.2 mm, 314 parts, among them J1 TYPE-C-31-M12_13, J2 PAD_SQUARE_1MM, J3 PAD_SQUARE_1MM, J4 PAD_SQUARE_1MM, J5 PAD_SQUARE_1MM, J6 Conn_01x04, K1 SMD-SWITCH-TACTILE-SPST-NO_4P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, Q1 MUN5311DW1T1G, Q2 MUN5311DW1T1G, SW1 RotaryEncoder_Switch, SW10 W, SW11 S, SW12 X, SW13 L_CMD, SW14 E, SW15 D, SW16 C, SW17 R, SW18 F, SW19 V, SW2 ESC, SW20 FN_1, SW21 T, SW22 G, SW23 B, SW24 Y, SW25 H, SW26 N, SW27 SPACE, SW28 U, SW29 J, SW3 TAB, SW30 M, SW31 I, SW32 K, SW33 COMMA, SW34 R_CMD, SW35 O, SW36 L, SW37 PERIOD, SW38 P, SW39 SEMI_COLON, SW4 L_SHIFT, SW40 SLASH, SW41 R_ALT, SW42 HYPHEN, SW43 APOSTROPHE, SW44 R_SHIFT, SW45 R_CTRL, SW46 EQUALS, SW47 RETURN, SW48 FN_2, SW49 BCK_SPC, SW5 L_CTRL, SW50 7, SW51 4, SW52 1, SW53 0, SW54 8, SW55 5, SW56 2, SW57 00, SW58 9, SW59 6, SW6 Q, SW60 3, SW61 NUM_PER, SW62 MINUS, SW63 PLUS, SW64 ENTER, SW65 PAD_LOCK, SW7 A, SW8 Z, SW9 L_ALT, U1 STM32F411CEU6, U2 SRV05-4, U3 SN74LV1T34DCKR, U4 AAP2967-33VIR1, U5 MB85RS64PNF-G-JNERE1, U6 SN74LV1T34DCKR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

Commit message: Wiring in USB and MCU
Parts:
- H1, H2, H3, H4, H5: footprint MountingHole:MountingHole_3.2mm_M3 -> MountingHole:MountingHole_2.2mm_M2
- H6: footprint MountingHole:MountingHole_3.2mm_M3_Pad -> MountingHole:MountingHole_2.2mm_M2_DIN965_Pad
- J2, J3, J4, J5: moved to F.Cu
- moved H1 351.5 mm to (373.0, 110.6)
- moved H6 331.9 mm to (373.0, 148.7)
- moved H2 197.2 mm to (220.6, 110.6)
- moved H3 189.2 mm to (230.2, 148.3)
- moved H5 80.7 mm to (49.1, 110.6)
- moved H4 48.7 mm to (53.9, 148.7)
- moved J4 41.9 mm to (306.8, 142.2), turned to 0 degrees
- moved U3 41.0 mm to (313.9, 133.1), turned to 0 degrees
- moved C1 39.4 mm to (301.8, 145.0), turned to 0 degrees
- moved J3 38.9 mm to (305.1, 138.9), turned to 0 degrees
- moved J5 37.8 mm to (308.6, 140.2), turned to 0 degrees
- moved D2 33.9 mm to (302.4, 149.4), turned to 0 degrees
- moved R5 32.3 mm to (311.4, 146.3), turned to -90 degrees
- moved R1 32.1 mm to (299.7, 143.5)
- moved R4 31.9 mm to (302.7, 150.6)
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Routing:
- net +3.3V: track 4.96 -> 90.0 mm, vias 0 -> 4
- net GND: track 136.9 -> 161.4 mm, vias 135 -> 150
- net /BOOT0: track 0.00 -> 11.3 mm, vias 0 -> 1
- net Net-(D5-Pad2): track 12.2 -> 1.27 mm, vias 2 -> 0
- net /NRST: track 0.00 -> 8.72 mm, vias 0 -> 2
- net /SwitchPin: track 0.00 -> 6.53 mm
- net Net-(D4-Pad1): track 10.6 -> 4.14 mm, vias 2 -> 0
- net VBUS: track 23.0 -> 16.8 mm
- net /F0: track 0.00 -> 4.90 mm
- net /F1: track 0.00 -> 4.68 mm
- net COL0: track 412.8 -> 408.2 mm
- net /D+: track 9.43 -> 6.61 mm
- net /D-: track 8.86 -> 11.2 mm
- net /VCAP_1: track 0.00 -> 2.18 mm
- net Net-(D1-Pad+): track 0.00 -> 1.56 mm
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Other:
- rule pad_to_mask_clearance: 0 -> 0.05
