File: The-GarlicBoard-2.kicad_sch (KiCad schematic)
At the start: 27 parts

Commit message: More schematic updates, added three LDO options
Parts:
- removed OL?: OLED, symbol kbd:OLED
- added C?: C, symbol Device:C
- added C? (x4): 1μF, symbol Device:C
- added C? (x4): 100nF, symbol Device:C
- added C?: (no value), symbol Device:C
- added D?: (no value), symbol Diode:BAT54C
- added OL?: OLED, symbol GarlicBoard-2-Parts:OLED
- added U?: AP7343-X2, symbol GarlicBoard-2-Parts:AP7343-X2
- added U?: AP7343-SOT25, symbol GarlicBoard-2-Parts:AP7343-SOT25
- C? (x2): value (none) -> 1μF/X7R
- C?: value (none) -> 22nF
- U?: value (none) -> RT9193
Connections:
- net +3V3: now also C?.1, C?.1, C?.1, C?.1, C?.1, C?.1, D?.2, U?.1 (VOUT), U?.5 (VOUT); no longer U?.3 (EN)
- net +5V: now also U?.3 (EN), C?.2, C?.2, OL?.3 (VCC), U?.1 (VIN), U?.3 (EN), U?.3 (EN), U?.4 (VIN)
- net GND: now also C?.1, C?.1, C?.2, C?.2, C?.2, C?.2, C?.2, C?.2, C?.2, C?.2, OL?.4 (GND), U?.2 (GND), U?.2 (GND), U?.5 (EP)
- net SCL: now also OL?.2 (SCL)
- net SDA: now also OL?.1 (SDA)
- net VBAT: now also C?.1, D?.3
- net VREF+: now reaches L?.1, U?.9 (VDDA)
- net VREF+: now also C?.1
- new net VB: D?.1
- no-connect marks 2 -> 3
Other:
- note added: "LDO AP7343 - SOT25"
- note added: "LDO AP7343 - X2-DFN1010-4"
- note added: "LDO RT9193"
- note added: "POWER SUPPLY"
- note added: "RTC CIRCUIT"
- note added: "STILL NEED C VALUE"
- note added: "USB JST TO HUB BOARD"
- moved on the sheet: C?, J?, L?, U?

Commit message: Updated mainboard schematic
Parts:
- removed C?: C, symbol Device:C
- removed C? (x2): 1μF/X7R, symbol Device:C
- removed C? (x4): 1μF, symbol Device:C
- removed C?: 22nF, symbol Device:C
- removed C? (x4): 100nF, symbol Device:C
- removed C?: 0.1uF, symbol Device:C
- removed C?: (no value), symbol Device:C
- removed D?: SMF9.0CA, acheron_Components:D_SOD-123_Bidirectional, symbol Device:D_TVS
- removed D?: (no value), symbol Diode:BAT54C
- removed F?: ASMD1206-150, Fuse:Fuse_1206_3216Metric, symbol Device:Polyfuse
- removed G?: Unified-Daughterboard-Logo, Unified-Daughterboard-Logo:Unified-Daughterboard-Logo.pretty, symbol Mechanical:MountingHole
- removed G?: Unified-Daughterboard-Name, Unified-Daughterboard-Logo:Unified-Daughterboard-Name.pretty, symbol Mechanical:MountingHole
- removed J?: SM04B-SRSS-TB(LF)(SN), random-keyboard-parts:JST-SR-4, symbol Connector_Generic:Conn_01x04
- removed J?: TYPE-C-31-M12_13, acheron_Connectors:TYPE-C-31-M-12, symbol Unified-Daughterboard-rescue:TYPE-C-31-M12_13-acheronSymbols
- removed L?: 60R@100MHz, Inductor_SMD:L_1206_3216Metric, symbol Unified-Daughterboard-rescue:L_Core_Ferrite-Device
- removed L?: 1KΩ 100Mhz ±10%, symbol Device:L_Iron
- removed LED?: YS-SK6812MINI-E, symbol kbd:YS-SK6812MINI-E
- removed MH? (x4): Mount-M2, random-keyboard-parts:Generic-Mounthole, symbol Connector_Generic:Conn_01x01
- removed R? (x2): 4.7k, symbol Device:R
- removed R? (x2): 5.1k, Resistors_SMD:R_0603, symbol Device:R_Small
- removed U?: STM32F411CCUx, Package_DFN_QFN:QFN-48-1EP_7x7mm_P0.5mm_EP5.6x5.6mm, symbol MCU_ST_STM32F4:STM32F411CCUx
- removed U?: TPD4E05U06DQAR, acheron_Components:USON-10_2.5x1.0mm_P0.5mm, symbol Unified-Daughterboard-rescue:TPD4E05U06DQAR-acheronSymbols
- removed U?: AP7343-X2, symbol GarlicBoard-2-Parts:AP7343-X2
- removed U?: RT9193, symbol GarlicBoard-2-Parts:RT9193
- removed U?: AP7343-SOT25, symbol GarlicBoard-2-Parts:AP7343-SOT25
- removed U?: W25Q32JVSS, Package_SO:SOIC-8_5.23x5.23mm_P1.27mm, symbol Memory_Flash:W25Q32JVSS
- added C? (x2): cap_4.7uF_10v_0402, Bonsai_C4:C_0402_1005Metric, symbol Bonsai_C4:cap_4.7uF_10v_0402
- added C? (x2): cap_1uF_10v_0402, Bonsai_C4:C_0402_1005Metric, symbol Bonsai_C4:cap_1uF_10v_0402
- added C? (x7): cap_100nF_16v_0402, Bonsai_C4:C_0402_1005Metric, symbol Bonsai_C4:cap_100nF_16v_0402
- added C? (x2): cap_20pF_50v_0402, Bonsai_C4:C_0402_1005Metric, symbol Bonsai_C4:cap_20pF_50v_0402
- added C?: cap_10uF_10v_0402, Bonsai_C4:C_0402_1005Metric, symbol Bonsai_C4:cap_10uF_10v_0402
- added D? (x65): D, symbol Device:D
- added D?: SMD-LED-WHITE_0402_, Bonsai_C4:LED_0402, symbol Bonsai_C4:SMD-LED-WHITE_0402_
- added D?: 1N4148, Bonsai_C4:D_SOD-523, symbol Bonsai_C4:1N4148
- added H?: (no value), symbol Mechanical:MountingHole
- added H? (x5): MH, symbol Mechanical:MountingHole
- added J?: Conn_01x04, symbol Connector_Generic:Conn_01x04
- added J? (x3): PAD_SQUARE_1MM, Bonsai_C4:PAD_SQUARE_1MM, symbol Bonsai_C4:PAD_SQUARE_1MM
- added K?: SMD-SWITCH-TACTILE-SPST-NO_4P-3.0MMx2.6MM_, Bonsai_C4:SW4-SMD-3.0X2.6X0.7MM, symbol Bonsai_C4:SMD-SWITCH-TACTILE-SPST-NO_4P-3.0MMx2.6MM_
- added LED? (x64): SK6812, symbol kbd:YS-SK6812MINI-E
- added Q? (x2): MUN5311DW1T1G, Bonsai_C4:SOT-363_SC-70-6_SC-88, symbol Bonsai_C4:MUN5311DW1T1G
- added R? (x2): r_100k_0402_1p, Bonsai_C4:R_0402_1005Metric, symbol Bonsai_C4:r_100k_0402_1p
- added R? (x2): 4.7k, symbol Device:R
- added R? (x2): r_75_0402_1p, Bonsai_C4:R_0402_1005Metric, symbol Bonsai_C4:r_75_0402_1p
- added R?: r_470_0402_1p, Bonsai_C4:R_0402_1005Metric, symbol Bonsai_C4:r_470_0402_1p
- added SW? (x64): SW_PUSH, symbol kbd:SW_PUSH
- added SW?: RotaryEncoder_Switch, symbol Device:RotaryEncoder_Switch
- added U? (x2): SN74LV1T34DCKR, Bonsai_C4:SOT-353_SC-70-5, symbol Bonsai_C4:SN74LV1T34DCKR
- added U?: MB85RS64PNF-G-JNERE1, Bonsai_C4:SOP-8_3.9x4.9mm_P1.27mm, symbol Bonsai_C4:MB85RS64PNF-G-JNERE1
- added U?: W25Q128JVSIQ, Bonsai_C4:SOIC-8_5.23x5.23mm_P1.27mm, symbol Bonsai_C4:W25Q128JVSIQ
- added U?: AAP2967-33VIR1, Bonsai_C4:SOT-23-5, symbol Bonsai_C4:AAP2967-33VIR1
- added U?: STM32F411CEU6, Bonsai_C4:QFN-48-1EP_7x7mm_P0.5mm_EP5.6x5.6mm_ThermalVias, symbol Bonsai_C4:STM32F411CEU6
- added Y?: SMD-CRYSTAL-8MHZ-20PF-10PPM_2P-5.0X3.2MM_, Bonsai_C4:X2-SMD-5.0X3.2X1.3MM, symbol Bonsai_C4:SMD-CRYSTAL-8MHZ-20PF-10PPM_2P-5.0X3.2MM_
Connections:
- net VCC is gone; now on net +5V: J?.1 (Pin_1)
- net +3V3: now also C?.1, C?.1, C?.1, C?.1, C?.1, C?.1, C?.1, C?.1, J?.1 (Pin_1), K?.2 (A1), Q?.4 (E), R?.1, R?.1, R?.1, R?.1, U?.1 (VBAT), U?.24 (VDD), U?.3 (~{WP}), U?.36 (VDD), U?.48 (VDD), U?.5 (VCC), U?.5 (VOUT), U?.7 (~{HOLD}), U?.8 (VCC), U?.8 (VDD), U?.9 (VDDA)
- net +5V: now also C?.1, LED?.1 (VDD), LED?.1 (VDD), LED?.1 (VDD), LED?.1 (VDD), LED?.1 (VDD), LED?.1 (VDD), LED?.1 (VDD), LED?.1 (VDD), LED?.1 (VDD), LED?.1 (VDD), LED?.1 (VDD), LED?.1 (VDD), LED?.1 (VDD), LED?.1 (VDD), LED?.1 (VDD), LED?.1 (VDD), LED?.1 (VDD), LED?.1 (VDD), LED?.1 (VDD), LED?.1 (VDD), LED?.1 (VDD), LED?.1 (VDD), LED?.1 (VDD), LED?.1 (VDD), LED?.1 (VDD), LED?.1 (VDD), LED?.1 (VDD), LED?.1 (VDD), LED?.1 (VDD), LED?.1 (VDD), LED?.1 (VDD), LED?.1 (VDD), LED?.1 (VDD), LED?.1 (VDD), LED?.1 (VDD), LED?.1 (VDD), LED?.1 (VDD), LED?.1 (VDD), LED?.1 (VDD), LED?.1 (VDD), LED?.1 (VDD), LED?.1 (VDD), LED?.1 (VDD), LED?.1 (VDD), LED?.1 (VDD), LED?.1 (VDD), LED?.1 (VDD), LED?.1 (VDD), LED?.1 (VDD), LED?.1 (VDD), LED?.1 (VDD), LED?.1 (VDD), LED?.1 (VDD), LED?.1 (VDD), LED?.1 (VDD), LED?.1 (VDD), LED?.1 (VDD), LED?.1 (VDD), LED?.1 (VDD), LED?.1 (VDD), LED?.1 (VDD), LED?.1 (VDD), LED?.1 (VDD), LED?.1 (VDD), U?.1 (VIN), U?.3 (EN), U?.5 (VCC)
- net GND: now also C?.2, C?.2, C?.2, C?.2, C?.2, C?.2, C?.2, C?.2, C?.2, C?.2, C?.2, C?.2, C?.2, C?.2, J?.4 (Pin_4), LED?.3 (VSS), LED?.3 (VSS), LED?.3 (VSS), LED?.3 (VSS), LED?.3 (VSS), LED?.3 (VSS), LED?.3 (VSS), LED?.3 (VSS), LED?.3 (VSS), LED?.3 (VSS), LED?.3 (VSS), LED?.3 (VSS), LED?.3 (VSS), LED?.3 (VSS), LED?.3 (VSS), LED?.3 (VSS), LED?.3 (VSS), LED?.3 (VSS), LED?.3 (VSS), LED?.3 (VSS), LED?.3 (VSS), LED?.3 (VSS), LED?.3 (VSS), LED?.3 (VSS), LED?.3 (VSS), LED?.3 (VSS), LED?.3 (VSS), LED?.3 (VSS), LED?.3 (VSS), LED?.3 (VSS), LED?.3 (VSS), LED?.3 (VSS), LED?.3 (VSS), LED?.3 (VSS), LED?.3 (VSS), LED?.3 (VSS), LED?.3 (VSS), LED?.3 (VSS), LED?.3 (VSS), LED?.3 (VSS), LED?.3 (VSS), LED?.3 (VSS), LED?.3 (VSS), LED?.3 (VSS), LED?.3 (VSS), LED?.3 (VSS), LED?.3 (VSS), LED?.3 (VSS), LED?.3 (VSS), LED?.3 (VSS), LED?.3 (VSS), LED?.3 (VSS), LED?.3 (VSS), LED?.3 (VSS), LED?.3 (VSS), LED?.3 (VSS), LED?.3 (VSS), LED?.3 (VSS), LED?.3 (VSS), LED?.3 (VSS), LED?.3 (VSS), LED?.3 (VSS), LED?.3 (VSS), LED?.3 (VSS), Q?.1 (E), Q?.1 (E), Q?.3 (C), R?.2, SW?.C, U?.2 (GND), U?.23 (VSS), U?.3 (GND), U?.3 (GND), U?.35 (VSS), U?.4 (GND), U?.4 (VSS), U?.47 (VSS), U?.49 (EP), U?.8 (VSSA)
- net SCL: now also R?.2, U?.42 (PB6)
- net SDA: now also R?.2, U?.43 (PB7)
- net DA+ renamed DP
- net DP: now also U?.33 (PA12)
- net DA- renamed DN
- net DN: now also U?.32 (PA11)
- new net: D?.2 (A), SW?.1 (x64)
- new net: LED?.2 (DOUT), LED?.4 (DIN) (x63)
- new net: C?.1, D?.- (K), R?.1, U?.2
- new net: D?.+, R?.2
- new net: D?.-, Q?.4 (E)
- new net: Q?.6 (C), R?.1
- new net: D?.+ (A), R?.2
- new net A0_FRAM_CS: U?.1 (~{CS}), U?.10 (PA0)
- new net A10: R?.2, U?.2, U?.31 (PA10)
- new net A10_5V: LED?.4 (DIN), U?.4
- new net B12_FLASH_CS: U?.1 (~{CS}), U?.25 (PB12)
- new net B2: J?.1, Q?.5, R?.2, U?.20 (PB2)
- new net B3_SCK: U?.39 (PB3), U?.6 (CLK), U?.6 (SCK)
- new net B4_MISO: U?.2 (DO(IO1)), U?.2 (SO), U?.40 (PB4)
- new net B5_MOSI: U?.41 (PB5), U?.5 (DI(IO0)), U?.5 (SI)
- new net BOOT0: J?.1, Q?.2 (B), U?.4, U?.44 (BOOT0)
- new net C15: U?.4 (PC15)
- new net COL0: SW?.2, SW?.2, SW?.2, SW?.2, SW?.2, SW?.2, SW?.2, SW?.2, U?.11 (PA1)
- new net COL1: SW?.2, SW?.2, SW?.2, SW?.2, SW?.2, SW?.2, SW?.2, U?.12 (PA2)
- new net COL2: SW?.2, SW?.2, SW?.2, SW?.2, SW?.2, SW?.2, SW?.2, U?.13 (PA3)
- new net COL3: SW?.2, SW?.2, SW?.2, SW?.2, SW?.2, SW?.2, SW?.2, U?.14 (PA4)
- new net COL4: SW?.2, SW?.2, SW?.2, SW?.2, SW?.2, SW?.2, SW?.2, U?.15 (PA5)
- new net COL5: SW?.2, SW?.2, SW?.2, SW?.2, SW?.2, SW?.2, SW?.2, SW?.2, U?.16 (PA6)
- new net COL6: SW?.2, SW?.2, SW?.2, SW?.2, SW?.S2, U?.17 (PA7)
- new net COL7: SW?.2, SW?.2, SW?.2, SW?.2, SW?.2, SW?.2, SW?.2, SW?.2, U?.29 (PA8)
- new net COL8: SW?.2, SW?.2, SW?.2, SW?.2, SW?.2, SW?.2, SW?.2, SW?.2, U?.38 (PA15)
- new net DFU: Q?.5
- new net ENCSW1: D?.2 (A), SW?.S1
- new net ENC_A: SW?.A, U?.2 (PC13)
- new net ENC_B: SW?.B, U?.3 (PC14)
- new net F0: C?.1, U?.5 (PH0-OSC_IN), Y?.1
- new net F1: C?.1, U?.6 (PH0-OSC_OUT), Y?.2
- new net NRST: C?.1, J?.1, Q?.6 (C), U?.7 (NRST)
- new net ROW0: D?.1 (K), D?.1 (K), D?.1 (K), D?.1 (K), D?.1 (K), D?.1 (K), D?.1 (K), D?.1 (K), D?.1 (K), U?.18 (PB0)
- new net ROW1: D?.1 (K), D?.1 (K), D?.1 (K), D?.1 (K), D?.1 (K), D?.1 (K), D?.1 (K), D?.1 (K), D?.1 (K), U?.19 (PB1)
- new net ROW2: D?.1 (K), D?.1 (K), D?.1 (K), D?.1 (K), D?.1 (K), D?.1 (K), D?.1 (K), D?.1 (K), U?.45 (PB8)
- new net ROW3: D?.1 (K), D?.1 (K), D?.1 (K), D?.1 (K), D?.1 (K), D?.1 (K), D?.1 (K), D?.1 (K), D?.1 (K), U?.46 (PB9)
- new net ROW4: D?.1 (K), D?.1 (K), D?.1 (K), D?.1 (K), D?.1 (K), D?.1 (K), D?.1 (K), D?.1 (K), D?.1 (K), U?.21 (PB10)
- new net ROW5: D?.1 (K), D?.1 (K), D?.1 (K), D?.1 (K), D?.1 (K), D?.1 (K), D?.1 (K), D?.1 (K), D?.1 (K), U?.26 (PB13)
- new net ROW6: D?.1 (K), D?.1 (K), D?.1 (K), D?.1 (K), D?.1 (K), D?.1 (K), D?.1 (K), D?.1 (K), U?.27 (PB14)
- new net ROW7: D?.1 (K), D?.1 (K), D?.1 (K), D?.1 (K), U?.28 (PB15)
- new net SWCLK: J?.3 (Pin_3), U?.37 (PA14)
- new net SWDIO: J?.2 (Pin_2), U?.34 (PA13)
- new net SwitchPin: K?.4 (B1), Q?.2 (B), Q?.3 (C), R?.1
- new net VCAP_1: C?.1, U?.22 (VCAP_1)
- no-connect marks 3 -> 4
Other:
- added sheet UNIFIED PORT (unified port.kicad_sch)
- added sheet USB HUB (USB HUB.kicad_sch)
- note added: "1mm square pads on back"
- note added: "5V to drive WS2812"
- note added: "A10 TO RGB LED STRAND"
- note added: "BOOT"
- note added: "BOOT1"
- note added: "CRYSTAL"
- note added: "EMERGENCY PADS"
- note added: "FRAM AND FLASH"
- note added: "KEYBOARD INTERFACE"
- note added: "LDO"
- note added: "MCU"
- note added: "MOUNTING HOLES"
- note added: "RESET CIRCUIT"
- note added: "RGB STRAND"
- note added: "ROTARY ENCODER"
- note added: "SWITCH MATRIX"
- note added: "TO RGB STRAND"
- note removed: "CONNECTOR AND SHIELD UNIFIED"
- note removed: "ESD"
- note removed: "LDO AP7343 - SOT25"
- note removed: "LDO AP7343 - X2-DFN1010-4"
- note removed: "LDO RT9193"
- note removed: "MISC"
- note removed: "MOUNTING"
- note removed: "RTC CIRCUIT"
- note removed: "SERIAL FLASH"
- note removed: "STILL NEED C VALUE"
- moved on the sheet: J?, OL?

Commit message: More schematic updates
Parts:
- added C? (x134): 0.1uF, symbol Device:C
- added C? (x2): (no value), symbol Device:C
- added LED? (x136): SK6812, symbol kbd:YS-SK6812MINI-E
- added R? (x2): 4.7k, symbol Device:R
- H?: value (none) -> MH
Connections:
- net +3V3: now also R?.1, R?.1
- net ENC_A: now also R?.2
- net ENC_B: now also R?.2
- net GND: now also C?.2, C?.2, C?.2, C?.2, C?.2, C?.2, C?.2, C?.2, C?.2, C?.2, C?.2, C?.2, C?.2, C?.2, C?.2, C?.2, C?.2, C?.2, C?.2, C?.2, C?.2, C?.2, C?.2, C?.2, C?.2, C?.2, C?.2, C?.2, C?.2, C?.2, C?.2, C?.2, C?.2, C?.2, C?.2, C?.2, C?.2, C?.2, C?.2, C?.2, C?.2, C?.2, C?.2, C?.2, C?.2, C?.2, C?.2, C?.2, C?.2, C?.2, C?.2, C?.2, C?.2, C?.2, C?.2, C?.2, C?.2, C?.2, C?.2, C?.2, C?.2, C?.2, C?.2, C?.2, C?.2, C?.2, C?.2, C?.2, C?.2, C?.2, C?.2, C?.2, C?.2, C?.2, C?.2, C?.2, C?.2, C?.2, C?.2, C?.2, C?.2, C?.2, C?.2, C?.2, C?.2, C?.2, C?.2, C?.2, C?.2, C?.2, C?.2, C?.2, C?.2, C?.2, C?.2, C?.2, C?.2, C?.2, C?.2, C?.2, C?.2, C?.2, C?.2, C?.2, C?.2, C?.2, C?.2, C?.2, C?.2, C?.2, C?.2, C?.2, C?.2, C?.2, C?.2, C?.2, C?.2, C?.2, C?.2, C?.2, C?.2, C?.2, C?.2, C?.2, C?.2, C?.2, C?.2, C?.2, C?.2, C?.2, C?.2, C?.2, C?.2, C?.2, C?.2, C?.2
- new net: C?.1, LED?.1 (VDD) (x136)
- new net: LED?.2 (DOUT), LED?.4 (DIN) (x21)
- no-connect marks 4 -> 5
Other:
- note added: "May 1, 2022"
- note added: "The GarlicBoard 2"
- note added: "The GarlicBoard 2 Thomas Meyer a.k.a. stiligFox"
- moved on the sheet: R?

Commit message: First Major Update of 2023
Major updates to schematics and first revisions of PCB layout
Parts:
- removed C? (x70): 0.1uF, symbol Device:C
- removed C? (x2): cap_1uF_10v_0402, Bonsai_C4:C_0402_1005Metric, symbol Bonsai_C4:cap_1uF_10v_0402
- removed C? (x2): (no value), symbol Device:C
- removed D?: 1N4148, Bonsai_C4:D_SOD-523, symbol Bonsai_C4:1N4148
- removed H?: MH, symbol Mechanical:MountingHole
- removed J?: SM04B-SRSS-TB(LF)(SN), random-keyboard-parts:JST-SR-4, symbol Connector_Generic:Conn_01x04
- removed K?: SMD-SWITCH-TACTILE-SPST-NO_4P-3.0MMx2.6MM_, Bonsai_C4:SW4-SMD-3.0X2.6X0.7MM, symbol Bonsai_C4:SMD-SWITCH-TACTILE-SPST-NO_4P-3.0MMx2.6MM_
- removed LED? (x136): SK6812, symbol kbd:YS-SK6812MINI-E
- removed U?: AAP2967-33VIR1, Bonsai_C4:SOT-23-5, symbol Bonsai_C4:AAP2967-33VIR1
- added C18, C23: cap_1uF_10v_0402, Bonsai_C4:C_0402_1005Metric, symbol Bonsai_C4:cap_1uF_10v_0402
- added D2: 1N4148WT, Diode_SMD:D_SOD-523, symbol Diode:1N4148WT
- added D3: SMF5.0A, Bonsai_C4:D_SOD-123FL, symbol Bonsai_C4:SMF5.0A
- added D4, D5: PMEG2010AEB, Bonsai_C4:D_SOD-523, symbol Bonsai_C4:PMEG2010AEB
- added F1: SMD-PPTC-500MA_0805_, Bonsai_C4:F0805, symbol Bonsai_C4:SMD-PPTC-500MA_0805_
- added FB1: fb_0402_26ohm, Bonsai_C4:R_0402_1005Metric, symbol Bonsai_C4:fb_0402_26ohm
- added H6: MH_P, MountingHole:MountingHole_3.2mm_M3_Pad, symbol Mechanical:MountingHole_Pad
- added J1: TYPE-C-31-M12_13, Bonsai_C4:TYPE-C-31-M-12, symbol Bonsai_C4:TYPE-C-31-M12_13
- added J2: PAD_SQUARE_1MM, Bonsai_C4:PAD_SQUARE_1MM, symbol Bonsai_C4:PAD_SQUARE_1MM
- added K1: SMD-SWITCH-TACTILE-SPST-NO_4P-2.7MMx3.0MM_, Bonsai_C4:SW4-SMD-2.7X3.0X1.4MM, symbol Bonsai_C4:SMD-SWITCH-TACTILE-SPST-NO_4P-2.7MMx3.0MM_
- added R2, R3: 5.1k, Keebio-Parts:R_0402, symbol Device:R_Small
- added U2: SRV05-4, Bonsai_C4:SOT-23-6, symbol Bonsai_C4:SRV05-4
- added U4: AAP2967-33VIR1, Bonsai_C4:SOT-23-5, symbol Bonsai_C4:AAP2967-33VIR1
- C11, C12, C13, C14, C15, C16, C17, C19, C2, C20, C21, C22, C24, C25, C26, C27, C28, C29, C3, C30, C32, C33, C34, C39, C4, C40, C41, C44, C45, C46, C47, C5, C51, C52, C53, C54, C55, C56, C57, C58, C59, C6, C60, C61, C62, C63, C64, C65, C66, C67, C68, C69, C7, C70, C71, C72, C73, C74, C75, C76, C77, C78, C8, C9: renamed from C?; footprint (none) -> Capacitor_SMD:C_0402_1005Metric
- D10, D11, D12, D13, D14, D15, D16, D17, D18, D19, D20, D21, D22, D23, D24, D25, D26, D27, D28, D29, D30, D31, D32, D33, D34, D35, D36, D37, D38, D39, D40, D41, D42, D43, D44, D45, D46, D47, D48, D49, D50, D51, D52, D53, D54, D55, D56, D57, D58, D59, D6, D60, D61, D62, D63, D64, D65, D66, D67, D68, D69, D7, D70, D8, D9: renamed from D?; footprint (none) -> Diode_SMD:D_0402_1005Metric
- H1, H2, H3, H4, H5: renamed from H?; footprint (none) -> MountingHole:MountingHole_3.2mm_M3
- J6: renamed from J?; footprint (none) -> Connector_JST:JST_XH_B4B-XH-A_1x04_P2.50mm_Vertical
- LED1, LED10, LED11, LED12, LED13, LED14, LED15, LED16, LED17, LED18, LED19, LED2, LED20, LED21, LED22, LED23, LED24, LED25, LED26, LED27, LED28, LED29, LED3, LED30, LED31, LED32, LED33, LED34, LED35, LED36, LED37, LED38, LED39, LED4, LED40, LED41, LED42, LED43, LED44, LED45, LED46, LED47, LED48, LED49, LED5, LED50, LED51, LED52, LED53, LED54, LED55, LED56, LED57, LED58, LED59, LED6, LED60, LED61, LED62, LED63, LED64, LED7, LED8, LED9: renamed from LED?; footprint (none) -> Keebio-Parts:SK6812-MINI-E
- OL1: renamed from OL?; footprint (none) -> kbd:OLED_v2
- R10, R7, R8, R9: renamed from R?; footprint (none) -> Bonsai_C4:R_0402_1005Metric
- SW1: renamed from SW?; footprint (none) -> Keebio-Parts:RotaryEncoder_EC11
- SW10: renamed from SW?; value SW_PUSH -> W; footprint (none) -> MX_Hotswap:MX-Hotswap-1U
- SW11: renamed from SW?; value SW_PUSH -> S; footprint (none) -> MX_Hotswap:MX-Hotswap-1U
- SW12: renamed from SW?; value SW_PUSH -> X; footprint (none) -> MX_Hotswap:MX-Hotswap-1U
- SW13: renamed from SW?; value SW_PUSH -> L_CMD; footprint (none) -> MX_Hotswap:MX-Hotswap-1.25U
- SW14: renamed from SW?; value SW_PUSH -> E; footprint (none) -> MX_Hotswap:MX-Hotswap-1U
- SW15: renamed from SW?; value SW_PUSH -> D; footprint (none) -> MX_Hotswap:MX-Hotswap-1U
- SW16: renamed from SW?; value SW_PUSH -> C; footprint (none) -> MX_Hotswap:MX-Hotswap-1U
- SW17: renamed from SW?; value SW_PUSH -> R; footprint (none) -> MX_Hotswap:MX-Hotswap-1U
- SW18: renamed from SW?; value SW_PUSH -> F; footprint (none) -> MX_Hotswap:MX-Hotswap-1U
- SW19: renamed from SW?; value SW_PUSH -> V; footprint (none) -> MX_Hotswap:MX-Hotswap-1U
- SW2: renamed from SW?; value SW_PUSH -> ESC; footprint (none) -> MX_Hotswap:MX-Hotswap-1U
- SW20: renamed from SW?; value SW_PUSH -> FN_1; footprint (none) -> MX_Hotswap:MX-Hotswap-2.75U
- SW21: renamed from SW?; value SW_PUSH -> T; footprint (none) -> MX_Hotswap:MX-Hotswap-1U
- SW22: renamed from SW?; value SW_PUSH -> G; footprint (none) -> MX_Hotswap:MX-Hotswap-1U
- SW23: renamed from SW?; value SW_PUSH -> B; footprint (none) -> MX_Hotswap:MX-Hotswap-1U
- SW24: renamed from SW?; value SW_PUSH -> Y; footprint (none) -> MX_Hotswap:MX-Hotswap-1U
- SW25: renamed from SW?; value SW_PUSH -> H; footprint (none) -> MX_Hotswap:MX-Hotswap-1U
- SW26: renamed from SW?; value SW_PUSH -> N; footprint (none) -> MX_Hotswap:MX-Hotswap-1U
- SW27: renamed from SW?; value SW_PUSH -> SPACE; footprint (none) -> MX_Hotswap:MX-Hotswap-2.75U
- SW28: renamed from SW?; value SW_PUSH -> U; footprint (none) -> MX_Hotswap:MX-Hotswap-1U
- SW29: renamed from SW?; value SW_PUSH -> J; footprint (none) -> MX_Hotswap:MX-Hotswap-1U
- SW3: renamed from SW?; value SW_PUSH -> TAB; footprint (none) -> MX_Hotswap:MX-Hotswap-1.25U
- SW30: renamed from SW?; value SW_PUSH -> M; footprint (none) -> MX_Hotswap:MX-Hotswap-1U
- SW31: renamed from SW?; value SW_PUSH -> I; footprint (none) -> MX_Hotswap:MX-Hotswap-1U
- SW32: renamed from SW?; value SW_PUSH -> K; footprint (none) -> MX_Hotswap:MX-Hotswap-1U
- SW33: renamed from SW?; value SW_PUSH -> COMMA; footprint (none) -> MX_Hotswap:MX-Hotswap-1U
- SW34: renamed from SW?; value SW_PUSH -> R_CMD; footprint (none) -> MX_Hotswap:MX-Hotswap-1.25U
- SW35: renamed from SW?; value SW_PUSH -> O; footprint (none) -> MX_Hotswap:MX-Hotswap-1U
- SW36: renamed from SW?; value SW_PUSH -> L; footprint (none) -> MX_Hotswap:MX-Hotswap-1U
- SW37: renamed from SW?; value SW_PUSH -> PERIOD; footprint (none) -> MX_Hotswap:MX-Hotswap-1U
- SW38: renamed from SW?; value SW_PUSH -> P; footprint (none) -> MX_Hotswap:MX-Hotswap-1U
- SW39: renamed from SW?; value SW_PUSH -> SEMI_COLON; footprint (none) -> MX_Hotswap:MX-Hotswap-1U
- SW4: renamed from SW?; value SW_PUSH -> L_SHIFT; footprint (none) -> MX_Hotswap:MX-Hotswap-1.75U
- SW40: renamed from SW?; value SW_PUSH -> SLASH; footprint (none) -> MX_Hotswap:MX-Hotswap-1U
- SW41: renamed from SW?; value SW_PUSH -> R_ALT; footprint (none) -> MX_Hotswap:MX-Hotswap-1.25U
- SW42: renamed from SW?; value SW_PUSH -> HYPHEN; footprint (none) -> MX_Hotswap:MX-Hotswap-1U
- SW43: renamed from SW?; value SW_PUSH -> APOSTROPHE; footprint (none) -> MX_Hotswap:MX-Hotswap-1U
- SW44: renamed from SW?; value SW_PUSH -> R_SHIFT; footprint (none) -> MX_Hotswap:MX-Hotswap-2.25U
- SW45: renamed from SW?; value SW_PUSH -> R_CTRL; footprint (none) -> MX_Hotswap:MX-Hotswap-1.25U
- SW46: renamed from SW?; value SW_PUSH -> EQUALS; footprint (none) -> MX_Hotswap:MX-Hotswap-1U
- SW47: renamed from SW?; value SW_PUSH -> RETURN; footprint (none) -> MX_Hotswap:MX-Hotswap-1.75U
- SW48: renamed from SW?; value SW_PUSH -> FN_2; footprint (none) -> MX_Hotswap:MX-Hotswap-1U
- SW49: renamed from SW?; value SW_PUSH -> BCK_SPC; footprint (none) -> MX_Hotswap:MX-Hotswap-1U
- SW5: renamed from SW?; value SW_PUSH -> L_CTRL; footprint (none) -> MX_Hotswap:MX-Hotswap-1.25U
- SW50: renamed from SW?; value SW_PUSH -> 7; footprint (none) -> MX_Hotswap:MX-Hotswap-1U
- SW51: renamed from SW?; value SW_PUSH -> 4; footprint (none) -> MX_Hotswap:MX-Hotswap-1U
- SW52: renamed from SW?; value SW_PUSH -> 1; footprint (none) -> MX_Hotswap:MX-Hotswap-1U
- SW53: renamed from SW?; value SW_PUSH -> 0; footprint (none) -> MX_Hotswap:MX-Hotswap-1U
- SW54: renamed from SW?; value SW_PUSH -> 8; footprint (none) -> MX_Hotswap:MX-Hotswap-1U
- SW55: renamed from SW?; value SW_PUSH -> 5; footprint (none) -> MX_Hotswap:MX-Hotswap-1U
- SW56: renamed from SW?; value SW_PUSH -> 2; footprint (none) -> MX_Hotswap:MX-Hotswap-1U
- SW57: renamed from SW?; value SW_PUSH -> 00; footprint (none) -> MX_Hotswap:MX-Hotswap-1U
- SW58: renamed from SW?; value SW_PUSH -> 9; footprint (none) -> MX_Hotswap:MX-Hotswap-1U
- SW59: renamed from SW?; value SW_PUSH -> 6; footprint (none) -> MX_Hotswap:MX-Hotswap-1U
- SW6: renamed from SW?; value SW_PUSH -> Q; footprint (none) -> MX_Hotswap:MX-Hotswap-1U
- SW60: renamed from SW?; value SW_PUSH -> 3; footprint (none) -> MX_Hotswap:MX-Hotswap-1U
- SW61: renamed from SW?; value SW_PUSH -> NUM_PER; footprint (none) -> MX_Hotswap:MX-Hotswap-1U
- SW62: renamed from SW?; value SW_PUSH -> MINUS; footprint (none) -> MX_Hotswap:MX-Hotswap-1U
- SW63: renamed from SW?; value SW_PUSH -> PLUS; footprint (none) -> MX_Hotswap:MX-Hotswap-1U
- SW64: renamed from SW?; value SW_PUSH -> ENTER; footprint (none) -> MX_Hotswap:MX-Hotswap-1U
- SW65: renamed from SW?; value SW_PUSH -> PAD_LOCK; footprint (none) -> MX_Hotswap:MX-Hotswap-1U
- SW7: renamed from SW?; value SW_PUSH -> A; footprint (none) -> MX_Hotswap:MX-Hotswap-1U
- SW8: renamed from SW?; value SW_PUSH -> Z; footprint (none) -> MX_Hotswap:MX-Hotswap-1U
- SW9: renamed from SW?; value SW_PUSH -> L_ALT; footprint (none) -> MX_Hotswap:MX-Hotswap-1.25U
- gave numbers to parts that had none: 29
Connections:
- net +3V3: no longer C35.1, C36.1, C38.1, C42.1, C43.1, C49.1, C50.1, Q1.4 (E), R11.1, R5.1, U1.1 (VBAT), U1.24 (VDD), U1.36 (VDD), U1.48 (VDD), U1.9 (VDDA), U3.5 (VCC), U5.3 (~{WP}), U5.7 (~{HOLD}), U5.8 (VDD), U7.8 (VCC)
- net +5V: now also C18.1, D5.1 (K), U4.1 (VIN), U4.3 (EN); no longer OL1.3 (VCC), U6.5 (VCC)
- net A10_5V: now also LED1.4 (DIN)
- net COL0: now also U1.15 (PA5); no longer U1.11 (PA1)
- net COL1: now also U1.14 (PA4); no longer U1.12 (PA2)
- net COL3: now also U1.12 (PA2); no longer U1.14 (PA4)
- net COL4: now also U1.11 (PA1); no longer U1.15 (PA5)
- net DFU: now also J2.1
- net DN: now also U2.6 (IO4)
- net DP: now also U2.4 (IO3)
- net GND: now also LED1.3 (VSS), LED10.3 (VSS), LED11.3 (VSS), LED12.3 (VSS), LED13.3 (VSS), LED14.3 (VSS), LED15.3 (VSS), LED16.3 (VSS), LED17.3 (VSS), LED18.3 (VSS), LED19.3 (VSS), LED2.3 (VSS), LED20.3 (VSS), LED21.3 (VSS), LED22.3 (VSS), LED23.3 (VSS), LED24.3 (VSS), LED25.3 (VSS), LED26.3 (VSS), LED27.3 (VSS), LED28.3 (VSS), LED29.3 (VSS), LED3.3 (VSS), LED30.3 (VSS), LED31.3 (VSS), LED32.3 (VSS), LED33.3 (VSS), LED34.3 (VSS), LED35.3 (VSS), LED36.3 (VSS), LED37.3 (VSS), LED38.3 (VSS), LED39.3 (VSS), LED4.3 (VSS), LED40.3 (VSS), LED41.3 (VSS), LED42.3 (VSS), LED43.3 (VSS), LED44.3 (VSS), LED45.3 (VSS), LED46.3 (VSS), LED47.3 (VSS), LED48.3 (VSS), LED49.3 (VSS), LED5.3 (VSS), LED50.3 (VSS), LED51.3 (VSS), LED52.3 (VSS), LED53.3 (VSS), LED54.3 (VSS), LED55.3 (VSS), LED56.3 (VSS), LED57.3 (VSS), LED58.3 (VSS), LED59.3 (VSS), LED6.3 (VSS), LED60.3 (VSS), LED61.3 (VSS), LED62.3 (VSS), LED63.3 (VSS), LED64.3 (VSS), LED7.3 (VSS), LED8.3 (VSS), LED9.3 (VSS), C18.2, C23.2, D3.2 (A2), FB1.2, H6.1, J1.A1 (GND), J1.B1 (GND), R2.2, R3.2, U2.2 (VN), U4.2 (GND)
- net SwitchPin: now also K1.4 (B1)
- net VCC: now reaches C44.1, LED33.1 (VDD)
- net VCC: now also C11.1, C12.1, C13.1, C14.1, C15.1, C16.1, C17.1, C19.1, C2.1, C20.1, C21.1, C22.1, C24.1, C25.1, C26.1, C27.1, C28.1, C29.1, C3.1, C30.1, C32.1, C33.1, C34.1, C39.1, C4.1, C40.1, C41.1, C45.1, C46.1, C47.1, C5.1, C51.1, C52.1, C53.1, C54.1, C55.1, C56.1, C57.1, C58.1, C59.1, C6.1, C60.1, C61.1, C62.1, C63.1, C64.1, C65.1, C66.1, C67.1, C68.1, C69.1, C7.1, C70.1, C71.1, C72.1, C73.1, C74.1, C75.1, C76.1, C77.1, C78.1, C8.1, C9.1, LED1.1 (VDD), LED10.1 (VDD), LED11.1 (VDD), LED12.1 (VDD), LED13.1 (VDD), LED14.1 (VDD), LED15.1 (VDD), LED16.1 (VDD), LED17.1 (VDD), LED18.1 (VDD), LED19.1 (VDD), LED2.1 (VDD), LED20.1 (VDD), LED21.1 (VDD), LED22.1 (VDD), LED23.1 (VDD), LED24.1 (VDD), LED25.1 (VDD), LED26.1 (VDD), LED27.1 (VDD), LED28.1 (VDD), LED29.1 (VDD), LED3.1 (VDD), LED30.1 (VDD), LED31.1 (VDD), LED32.1 (VDD), LED34.1 (VDD), LED35.1 (VDD), LED36.1 (VDD), LED37.1 (VDD), LED38.1 (VDD), LED39.1 (VDD), LED4.1 (VDD), LED40.1 (VDD), LED41.1 (VDD), LED42.1 (VDD), LED43.1 (VDD), LED44.1 (VDD), LED45.1 (VDD), LED46.1 (VDD), LED47.1 (VDD), LED48.1 (VDD), LED49.1 (VDD), LED5.1 (VDD), LED50.1 (VDD), LED51.1 (VDD), LED52.1 (VDD), LED53.1 (VDD), LED54.1 (VDD), LED55.1 (VDD), LED56.1 (VDD), LED57.1 (VDD), LED58.1 (VDD), LED59.1 (VDD), LED6.1 (VDD), LED60.1 (VDD), LED61.1 (VDD), LED62.1 (VDD), LED63.1 (VDD), LED64.1 (VDD), LED7.1 (VDD), LED8.1 (VDD), LED9.1 (VDD), OL1.3 (VCC), U6.5 (VCC)
- net at LED33.2 (DOUT): now also LED37.4 (DIN)
- net at LED33.4 (DIN): now also LED34.2 (DOUT)
- net at LED18.2 (DOUT): now also LED19.4 (DIN)
- net at LED18.4 (DIN): now also LED17.2 (DOUT)
- net at C10.1, R6.1, U3.2: now also D2.1 (K)
- net at LED53.2 (DOUT): now also LED57.4 (DIN)
- net at LED53.4 (DIN): now also LED54.2 (DOUT)
- net at LED41.2 (DOUT): now also LED44.4 (DIN)
- net at LED41.4 (DIN): now also LED42.2 (DOUT)
- net at LED24.2 (DOUT): now also LED25.4 (DIN)
- net at LED24.4 (DIN): now also LED23.2 (DOUT)
- net at LED13.2 (DOUT): now also LED16.4 (DIN)
- net at LED13.4 (DIN): now also LED14.2 (DOUT)
- net at LED52.2 (DOUT): now also LED56.4 (DIN)
- net at LED52.4 (DIN): now also LED51.2 (DOUT)
- net at LED14.4 (DIN): now also LED15.2 (DOUT)
- net at LED59.2 (DOUT): now also LED60.4 (DIN)
- net at LED59.4 (DIN): now also LED58.2 (DOUT)
- net at LED30.2 (DOUT): now also LED31.4 (DIN)
- net at LED30.4 (DIN): now also LED27.2 (DOUT)
- net at LED60.2 (DOUT): now also LED64.4 (DIN)
- net at LED34.4 (DIN): now also LED35.2 (DOUT)
- net at LED51.4 (DIN): now also LED50.2 (DOUT)
- net at LED47.2 (DOUT): now also LED49.4 (DIN)
- net at LED47.4 (DIN): now also LED48.2 (DOUT)
- net at LED21.2 (DOUT): now also LED20.4 (DIN)
- net at LED21.4 (DIN): now also LED22.2 (DOUT)
- net at LED36.2 (DOUT): now also LED35.4 (DIN)
- net at LED36.4 (DIN): now also LED32.2 (DOUT)
- net at R4.2: now also D2.2 (A)
- net at LED50.4 (DIN): now also LED49.2 (DOUT)
- net at LED46.2 (DOUT): now also LED48.4 (DIN)
- net at LED46.4 (DIN): now also LED45.2 (DOUT)
- net at LED23.4 (DIN): now also LED20.2 (DOUT)
- net at LED39.2 (DOUT): now also LED40.4 (DIN)
- net at LED39.4 (DIN): now also LED38.2 (DOUT)
- net at LED17.4 (DIN): now also LED16.2 (DOUT)
- net at LED43.2 (DOUT): now also LED42.4 (DIN)
- net at LED43.4 (DIN): now also LED40.2 (DOUT)
- net at LED57.2 (DOUT): now also LED58.4 (DIN)
- net at LED5.2 (DOUT): now also LED9.4 (DIN)
- net at LED5.4 (DIN): now also LED6.2 (DOUT)
- net at LED15.4 (DIN): now also LED12.2 (DOUT)
- net at LED9.2 (DOUT): now also LED10.4 (DIN)
- net at LED8.2 (DOUT): now also LED7.4 (DIN)
- net at LED26.2 (DOUT): now also LED29.4 (DIN)
- net at LED26.4 (DIN): now also LED25.2 (DOUT)
- net at LED27.4 (DIN): now also LED28.2 (DOUT)
- net at LED19.2 (DOUT): now also LED22.4 (DIN)
- net at LED28.4 (DIN): now also LED29.2 (DOUT)
- net at LED31.2 (DOUT): now also LED32.4 (DIN)
- net at LED56.2 (DOUT): now also LED55.4 (DIN)
- net at LED55.2 (DOUT): now also LED54.4 (DIN)
- net at LED37.2 (DOUT): now also LED38.4 (DIN)
- net at LED7.2 (DOUT): now also LED6.4 (DIN)
- net at LED10.2 (DOUT): now also LED11.4 (DIN)
- net at LED11.2 (DOUT): now also LED12.4 (DIN)
- net at LED64.2 (DOUT): now also LED63.4 (DIN)
- net at LED61.4 (DIN): now also LED62.2 (DOUT)
- net at LED62.4 (DIN): now also LED63.2 (DOUT)
- net at LED44.2 (DOUT): now also LED45.4 (DIN)
- net C15: no longer names the net of U1.4 (PC15)
- new net: D5.2 (A), F1.1
- new net: J1.A5 (CC1), R2.1
- new net: J1.B5 (CC2), R3.1
- new net: FB1.1, J1.S (SHIELD)
- new net: D4.1 (K), U2.5 (VP)
- new net +3.3V: C23.1, C35.1, C36.1, C38.1, C42.1, C43.1, C49.1, C50.1, K1.2 (A1), Q1.4 (E), R11.1, R5.1, U1.1 (VBAT), U1.24 (VDD), U1.36 (VDD), U1.48 (VDD), U1.9 (VDDA), U3.5 (VCC), U4.5 (VOUT), U5.3 (~{WP}), U5.7 (~{HOLD}), U5.8 (VDD), U7.8 (VCC)
- new net D+: J1.A6 (D+), J1.B6 (D+), U2.3 (IO2)
- new net D-: J1.A7 (D-), J1.B7 (D-), U2.1 (IO1)
- new net VBUS: D3.1 (A1), D4.2 (A), F1.2, J1.A4 (VBUS), J1.B4 (VBUS)
- no-connect marks 5 -> 9
Other:
- removed sheet UNIFIED PORT
- removed sheet USB HUB
- note added: "'"
- note added: "+"
- note added: ","
- note added: "-"
- note added: "."
- note added: "/"
- note added: "0"
- note added: "00"
- note added: "1"
- note added: "2"
- note added: "3"
- note added: "4"
- note added: "5"
- note added: "6"
- note added: "7"
- note added: "8"
- note added: "9"
- note added: ";"
- note added: "="
- note added: "A"
- note added: "B"
- note added: "BCK SPC"
- note added: "C"
- note added: "D"
- note added: "E"
- note added: "ENTER"
- note added: "ESC"
- note added: "F"
- note added: "FN_1"
- note added: "FN_2"
- note added: "G"
- note added: "H"
- note added: "I"
- note added: "J"
- note added: "K"
- note added: "L"
- note added: "L_ALT"
- note added: "L_CMD"
- note added: "L_CTRL"
- note added: "L_SHIFT"
- note added: "M"
- note added: "N"
- note added: "O"
- note added: "P"
- note added: "PAD LOCK"
- note added: "PERIOD"
- note added: "Q"
- note added: "R"
- note added: "RETURN"
- note added: "R_ALT"
- note added: "R_CMD"
- note added: "R_CTRL"
- note added: "R_SHIFT"
- note added: "S"
- note added: "SPACE"
- note added: "T"
- note added: "TAB"
- note added: "U"
- note added: "USB CONNECTOR AND ESD"
- note added: "V"
- note added: "W"
- note added: "X"
- note added: "Y"
- note added: "Z"
- note removed: "LDO"
- note removed: "The GarlicBoard 2 Thomas Meyer a.k.a. stiligFox"
- note removed: "USB JST TO HUB BOARD"
- moved on the sheet: C1, C10, C11, C12, C13, C14, C15, C16, C17, C19, C2, C20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

Commit message: Wiring in USB and MCU
Parts:
- H1, H2, H3, H4, H5: footprint MountingHole:MountingHole_3.2mm_M3 -> MountingHole:MountingHole_2.2mm_M2
- H6: footprint MountingHole:MountingHole_3.2mm_M3_Pad -> MountingHole:MountingHole_2.2mm_M2_DIN965_Pad
Changed lines of the file:
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@@
       (effects (font (size 0.75 0.75)) (justify right))
     )
-    (property "Footprint" "MountingHole:MountingHole_3.2mm_M3" (id 2) (at 176.53 127 0)
+    (property "Footprint" "MountingHole:MountingHole_2.2mm_M2" (id 2) (at 176.53 127 0)
       (effects (font (size 0.75 0.75)) hide)
     )
@@
       (effects (font (size 0.75 0.75)) (justify right))
     )
-    (property "Footprint" "MountingHole:MountingHole_3.2mm_M3" (id 2) (at 176.53 119.38 0)
+    (property "Footprint" "MountingHole:MountingHole_2.2mm_M2" (id 2) (at 176.53 119.38 0)
       (effects (font (size 0.75 0.75)) hide)
     )
@@
       (effects (font (size 0.75 0.75)) (justify right))
     )
-    (property "Footprint" "MountingHole:MountingHole_3.2mm_M3" (id 2) (at 185.42 111.76 0)
+    (property "Footprint" "MountingHole:MountingHole_2.2mm_M2" (id 2) (at 185.42 111.76 0)
       (effects (font (size 0.75 0.75)) hide)
     )
@@
       (effects (font (size 0.75 0.75)) (justify left))
     )
-    (property "Footprint" "MountingHole:MountingHole_3.2mm_M3_Pad" (id 2) (at 185.42 128.27 0)
+    (property "Footprint" "MountingHole:MountingHole_2.2mm_M2_DIN965_Pad" (id 2) (at 185.42 128.27 0)
       (effects (font (size 1.27 1.27)) hide)
     )
@@
       (effects (font (size 0.75 0.75)) (justify right))
     )
-    (property "Footprint" "MountingHole:MountingHole_3.2mm_M3" (id 2) (at 176.53 111.76 0)
+    (property "Footprint" "MountingHole:MountingHole_2.2mm_M2" (id 2) (at 176.53 111.76 0)
       (effects (font (size 0.75 0.75)) hide)
     )
@@
       (effects (font (size 0.75 0.75)) (justify right))
     )
-    (property "Footprint" "MountingHole:MountingHole_3.2mm_M3" (id 2) (at 185.42 119.38 0)
+    (property "Footprint" "MountingHole:MountingHole_2.2mm_M2" (id 2) (at 185.42 119.38 0)
       (effects (font (size 0.75 0.75)) hide)
     )
@@
     )
     (path "/d8879e99-6ea8-4aad-801b-670372e45d61"
-      (reference "H1") (unit 1) (value "MH") (footprint "MountingHole:MountingHole_3.2mm_M3")
+      (reference "H1") (unit 1) (value "MH") (footprint "MountingHole:MountingHole_2.2mm_M2")
     )
     (path "/74e6df63-f215-4717-9dc9-6a1372d09ad9"
-      (reference "H2") (unit 1) (value "MH") (footprint "MountingHole:MountingHole_3.2mm_M3")
+      (reference "H2") (unit 1) (value "MH") (footprint "MountingHole:MountingHole_2.2mm_M2")
     )
     (path "/66ec7ef8-6e02-4d84-84e6-c26f6d8627ba"
-      (reference "H3") (unit 1) (value "MH") (footprint "MountingHole:MountingHole_3.2mm_M3")
+      (reference "H3") (unit 1) (value "MH") (footprint "MountingHole:MountingHole_2.2mm_M2")
     )
     (path "/9e7c0309-8345-410f-bac9-c5c030aa0b1a"
-      (reference "H4") (unit 1) (value "MH") (footprint "MountingHole:MountingHole_3.2mm_M3")
+      (reference "H4") (unit 1) (value "MH") (footprint "MountingHole:MountingHole_2.2mm_M2")
     )
     (path "/fc280b87-5823-47e1-ab5d-936a43eec992"
-      (reference "H5") (unit 1) (value "MH") (footprint "MountingHole:MountingHole_3.2mm_M3")
+      (reference "H5") (unit 1) (value "MH") (footprint "MountingHole:MountingHole_2.2mm_M2")
     )
     (path "/ad682211-9ada-4a52-8238-a90e13011f8e"
-      (reference "H6") (unit 1) (value "MH_P") (footprint "MountingHole:MountingHole_3.2mm_M3_Pad")
+      (reference "H6") (unit 1) (value "MH_P") (footprint "MountingHole:MountingHole_2.2mm_M2_DIN965_Pad")
     )
     (path "/036da8b1-e7d7-45e4-acc3-e5ee8c3b6035"

Commit message: Final Updates
Parts:
- C48, C49, C50: footprint Bonsai_C4:C_0402_1005Metric -> Capacitor_SMD:C_0402_1005Metric
- D4, D5: footprint Bonsai_C4:D_SOD-523 -> Diode_SMD:D_SOD-523
- J6: footprint Connector_JST:JST_XH_B4B-XH-A_1x04_P2.50mm_Vertical -> Connector_PinHeader_2.54mm:PinHeader_1x04_P2.54mm_Vertical
- LED1, LED10, LED11, LED12, LED13, LED14, LED15, LED16, LED17, LED18, LED19, LED2, LED20, LED21, LED22, LED23, LED24, LED25, LED26, LED27, LED28, LED29, LED3, LED30, LED31, LED32, LED33, LED34, LED35, LED36, LED37, LED38, LED39, LED4, LED40, LED41, LED42, LED43, LED44, LED45, LED46, LED47, LED48, LED49, LED5, LED50, LED51, LED52, LED53, LED54, LED55, LED56, LED57, LED58, LED59, LED6, LED60, LED61, LED62, LED63, LED64, LED7, LED8, LED9: footprint Keebio-Parts:SK6812-MINI-E -> kbd:YS-SK6812MINI-E
- R10, R11, R4, R5, R6, R7, R8, R9: footprint Bonsai_C4:R_0402_1005Metric -> Resistor_SMD:R_0402_1005Metric
- U2: footprint Bonsai_C4:SOT-23-6 -> marbastlib-various:SOT-23-6-routable
Connections:
- net +3.3V is gone; now on net +3V3: C23.1, C35.1, C36.1, C38.1, C42.1, C43.1, C49.1, C50.1, K1.2 (A1), Q1.4 (E), R11.1, R5.1, U1.1 (VBAT), U1.24 (VDD), U1.36 (VDD), U1.48 (VDD), U1.9 (VDDA), U3.5 (VCC), U4.5 (VOUT), U5.3 (~{WP}), U5.7 (~{HOLD}), U5.8 (VDD), U7.8 (VCC)
- net VCC is gone; now on net +5V: C11.1, C12.1, C13.1, C14.1, C15.1, C16.1, C17.1, C19.1, C2.1, C20.1, C21.1, C22.1, C24.1, C25.1, C26.1, C27.1, C28.1, C29.1, C3.1, C30.1, C32.1, C33.1, C34.1, C39.1, C4.1, C40.1, C41.1, C44.1, C45.1, C46.1, C47.1, C5.1, C51.1, C52.1, C53.1, C54.1, C55.1, C56.1, C57.1, C58.1, C59.1, C6.1, C60.1, C61.1, C62.1, C63.1, C64.1, C65.1, C66.1, C67.1, C68.1, C69.1, C7.1, C70.1, C71.1, C72.1, C73.1, C74.1, C75.1, C76.1, C77.1, C78.1, C8.1, C9.1, LED1.1 (VDD), LED10.1 (VDD), LED11.1 (VDD), LED12.1 (VDD), LED13.1 (VDD), LED14.1 (VDD), LED15.1 (VDD), LED16.1 (VDD), LED17.1 (VDD), LED18.1 (VDD), LED19.1 (VDD), LED2.1 (VDD), LED20.1 (VDD), LED21.1 (VDD), LED22.1 (VDD), LED23.1 (VDD), LED24.1 (VDD), LED25.1 (VDD), LED26.1 (VDD), LED27.1 (VDD), LED28.1 (VDD), LED29.1 (VDD), LED3.1 (VDD), LED30.1 (VDD), LED31.1 (VDD), LED32.1 (VDD), LED33.1 (VDD), LED34.1 (VDD), LED35.1 (VDD), LED36.1 (VDD), LED37.1 (VDD), LED38.1 (VDD), LED39.1 (VDD), LED4.1 (VDD), LED40.1 (VDD), LED41.1 (VDD), LED42.1 (VDD), LED43.1 (VDD), LED44.1 (VDD), LED45.1 (VDD), LED46.1 (VDD), LED47.1 (VDD), LED48.1 (VDD), LED49.1 (VDD), LED5.1 (VDD), LED50.1 (VDD), LED51.1 (VDD), LED52.1 (VDD), LED53.1 (VDD), LED54.1 (VDD), LED55.1 (VDD), LED56.1 (VDD), LED57.1 (VDD), LED58.1 (VDD), LED59.1 (VDD), LED6.1 (VDD), LED60.1 (VDD), LED61.1 (VDD), LED62.1 (VDD), LED63.1 (VDD), LED64.1 (VDD), LED7.1 (VDD), LED8.1 (VDD), LED9.1 (VDD), OL1.3 (VCC), U6.5 (VCC)
- net COL7: now also U1.46 (PB9); no longer U1.29 (PA8)
- net COL8: now also U1.45 (PB8); no longer U1.38 (PA15)
- net D+: now also U1.33 (PA12), U2.6 (IO4); no longer U2.3 (IO2)
- net D-: now also U1.32 (PA11)
- net ROW0: now also U1.38 (PA15); no longer U1.18 (PB0)
- net ROW1: now also U1.28 (PB15); no longer U1.19 (PB1)
- net ROW2: now also U1.21 (PB10); no longer U1.45 (PB8)
- net ROW3: now also U1.19 (PB1); no longer U1.46 (PB9)
- net ROW4: now also U1.29 (PA8); no longer U1.21 (PB10)
- net ROW5: now also U1.27 (PB14); no longer U1.26 (PB13)
- net ROW6: now also U1.26 (PB13); no longer U1.27 (PB14)
- net ROW7: now also U1.18 (PB0); no longer U1.28 (PB15)
- removed net DN: U1.32 (PA11), U2.6 (IO4)
- net DP: no longer names the net of U2.4 (IO3)
- net DP: no longer U1.33 (PA12)
- no-connect marks 9 -> 11
Other:
- note added: "May 1, 2022 - Jan 4, 2023"
- note added: "The GarlicBoard"
- note added: "The GarlicBoard Thomas Meyer"
- note added: "v2.0_230104"
- note removed: "May 1, 2022"
- note removed: "The GarlicBoard 2"
